Commit message: experiment:：跑了graco数据集

File: config/robot.urdf.xacro (robot description, xacro)
@@ -2,5 +2,5 @@
 <robot name="lio" xmlns:xacro="http://tixiaoshan.github.io/">
   <xacro:property name="PI" value="3.1415926535897931" />
-  <link name="imu_link"></link>
+<!-- <link name="imu_link"></link>
   <link name="base_link"></link>
   <joint name="imu_joint" type="fixed">
@@ -8,16 +8,28 @@
     <child link="imu_link" />
     <origin xyz="0 0 0" rpy="0 0 0" />
-  </joint>
-  <link name="lidar_link"> </link>
+  </joint> -->
+  <!-- <link name="lidar_link"> </link>
   <joint name="lidar_joint" type="fixed">
     <parent link="base_link" />
     <child link="lidar_link" />
     <origin xyz="0 0 0" rpy="0 0 0" />
+  </joint> -->
+  <!-- <link name="gnss"></link>
+  <joint name="imu_joint" type="fixed">
+    <parent link="base_link"/>
+    <child link="gnss" /> <origin xyz="0 0 0" rpy="0 0 0" />
+  </joint> -->
+  <link name="base_link"/>
+  <link name="gnss"/>
+  <joint name="gnss_joint" type="fixed">
+    <parent link="base_link"/>
+    <child link="gnss"/>
+    <origin xyz="0 0 0" rpy="0 0 0"/>
   </joint>
-  <!-- <link name="navsat_link"> </link>
-  <joint name="navsat_joint" type="fixed">
+  <link name="velodyne"> </link>
+  <joint name="velodyne_joint" type="fixed">
     <parent link="base_link" />
-    <child link="navsat_link" />
+    <child link="velodyne" />
     <origin xyz="0 0 0" rpy="0 0 0" />
-  </joint> -->
+  </joint>
 </robot>

Commit message: 单机：成功

File: config/robot.urdf.xacro (robot description, xacro)
@@ -2,23 +2,11 @@
 <robot name="lio" xmlns:xacro="http://tixiaoshan.github.io/">
   <xacro:property name="PI" value="3.1415926535897931" />
-<!-- <link name="imu_link"></link>
-  <link name="base_link"></link>
+  <link name="base_link"/>
+  <link name="imu"/>
   <joint name="imu_joint" type="fixed">
     <parent link="base_link"/>
-    <child link="imu_link" />
-    <origin xyz="0 0 0" rpy="0 0 0" />
-  </joint> -->
-  <!-- <link name="lidar_link"> </link>
-  <joint name="lidar_joint" type="fixed">
-    <parent link="base_link" />
-    <child link="lidar_link" />
-    <origin xyz="0 0 0" rpy="0 0 0" />
-  </joint> -->
-  <!-- <link name="gnss"></link>
-  <joint name="imu_joint" type="fixed">
-    <parent link="base_link"/>
-    <child link="gnss" /> <origin xyz="0 0 0" rpy="0 0 0" />
-  </joint> -->
-  <link name="base_link"/>
+    <child link="imu"/>
+    <origin xyz="0 0 0" rpy="0 0 0"/>
+  </joint>
   <link name="gnss"/>
   <joint name="gnss_joint" type="fixed">
@@ -27,9 +15,15 @@
     <origin xyz="0 0 0" rpy="0 0 0"/>
   </joint>
-  <link name="velodyne"> </link>
+  <link name="livox"/>
+  <joint name="livox_joint" type="fixed">
+    <parent link="base_link"/>
+    <child link="livox"/>
+    <origin xyz="0 0 0" rpy="0 0 0"/>
+  </joint>
+  <link name="velodyne"/>
   <joint name="velodyne_joint" type="fixed">
-    <parent link="base_link" />
-    <child link="velodyne" />
-    <origin xyz="0 0 0" rpy="0 0 0" />
+    <parent link="base_link"/>
+    <child link="velodyne"/>
+    <origin xyz="0 0 0" rpy="0 0 0"/>
   </joint>
 </robot>

Commit message: 更新源码

File: config/robot.urdf.xacro (robot description, xacro)
@@ -27,3 +27,9 @@
     <origin xyz="0 0 0" rpy="0 0 0"/>
   </joint>
+    <link name="ouster"/>
+  <joint name="ouster_joint" type="fixed">
+    <parent link="base_link"/>
+    <child link="ouster"/>
+    <origin xyz="0 0 0" rpy="0 0 0"/>
+  </joint>
 </robot>
